Commit message: Checkpoint fix

File: barista_robot_description/urdf/barista_robot_model.urdf (robot description, URDF)
Before this commit: robot box_bot, 18 links, 17 joints
Joints:
- joint back_yaw_joint: origin xyz=-0.178 0 0 rpy=0 0 0 -> xyz=-0.1428 0 0 rpy=0 0 0
- joint front_yaw_joint: origin xyz=0.178 0 0 rpy=0 0 0 -> xyz=0.1428 0 0 rpy=0 0 0
- joint laser_scan_link_joint: origin xyz=0.160 0 0.155 rpy=0 0 0 -> xyz=0.1428 0 0.155 rpy=0 0 0
