Commit message: multiple-robots

File: barista_robot_description/urdf/barista_robot_model.urdf.xacro (robot description, xacro)
@@ -2,4 +2,6 @@
 <robot xmlns:xacro="http://www.ros.org/wiki/xacro" name="my_box_bot">
 <xacro:arg name="include_laser" default="true" />
+<xacro:arg name="robot_name" default="barista" />
+<xacro:arg name="use_controllers" default="false" />
 <xacro:include filename="$(find barista_robot_description)/urdf/caster_wheel.xacro" />
 <xacro:include filename="$(find barista_robot_description)/urdf/cup_holder_tray.xacro" />
@@ -29,5 +31,5 @@
             <cylinder length="0.155" radius="0.178"/>
         </geometry>
-        <material name="blue"/>
+        <material name="$(arg robot_color)"/>
     </visual>
     <collision>
@@ -55,5 +57,5 @@
 <xacro:cup_holder_tray parent="base_link"/>
 <xacro:if value="$(arg include_laser)">
-    <xacro:laser_scanner parent="chassis"/>
+    <xacro:laser_scanner parent="chassis" robot_name="$(arg robot_name)"/>
 </xacro:if>
 <!-- ============================================================ -->
@@ -64,5 +66,5 @@
     <plugin filename="gz-sim-joint-state-publisher-system"
             name="gz::sim::systems::JointStatePublisher">
-        <topic>/joint_states</topic>
+        <topic>/$(arg robot_name)/joint_states</topic>
         <update_rate>30</update_rate>
         <joint_name>joint_left_wheel</joint_name>
@@ -84,15 +86,16 @@
         <wheel_separation>0.1</wheel_separation>
         <wheel_radius>0.035</wheel_radius>
-        <topic>cmd_vel</topic>
+        <topic>/$(arg robot_name)/cmd_vel</topic>
         <publish_odom>true</publish_odom>
         <publish_odom_tf>true</publish_odom_tf>
         <publish_wheel_tf>true</publish_wheel_tf>
-        <odom_topic>odom</odom_topic>
-        <tf_topic>tf</tf_topic>
-        <frame_id>odom</frame_id>
-        <child_frame_id>base_link</child_frame_id>
+        <odom_topic>/$(arg robot_name)/odom</odom_topic>
+        <tf_topic>/$(arg robot_name)/tf</tf_topic>
+        <frame_id>$(arg robot_name)/odom</frame_id>
+        <child_frame_id>$(arg robot_name)/base_link</child_frame_id>
     </plugin>
 </gazebo>
 <!-- Enable Sensors in Gazebo Sim -->
+<!--
 <gazebo>
     <plugin filename="gz-sim-sensors-system" name="gz::sim::systems::Sensors">
@@ -100,3 +103,4 @@
     </plugin>
 </gazebo>
+-->
 </robot>

File: barista_robot_description/urdf/cup_holder_tray.xacro (robot description, xacro)
@@ -8,5 +8,5 @@
         <origin xyz="0 0 0" rpy="0 0 0"/>
         <geometry><cylinder length="0.090" radius="0.160"/></geometry>
-        <material name="blue"/>
+        <material name="$(arg robot_color)"/>
       </visual>
       <!--

File: barista_robot_description/urdf/laser_scanner.xacro (robot description, xacro)
@@ -5,5 +5,5 @@
        top. Includes the ros2_control hardware interface for both actuated
        joints and the gz gpu_lidar sensor plugin publishing on /scan. -->
-  <xacro:macro name="laser_scanner" params="parent">
+  <xacro:macro name="laser_scanner" params="parent robot_name:=barista use_ros2_control:=false">
     <link name="laser_scan_link">
       <visual>
@@ -95,5 +95,12 @@
       <plugin filename="gz_ros2_control-system"
               name="gz_ros2_control::GazeboSimROS2ControlPlugin">
-        <parameters>$(find my_box_bot_description)/config/controller_position.yaml</parameters>
+        <ros>
+          <namespace>/${robot_name}</namespace>
+          <!-- Some gz_ros2_control versions subscribe to the absolute
+               /robot_description topic even when namespaced; remap both
+               forms so each controller_manager gets its own robot. -->
+          <remapping>/robot_description:=/${robot_name}/robot_description</remapping>
+          <remapping>robot_description:=/${robot_name}/robot_description</remapping>
+        </ros>
       </plugin>
     </gazebo>
@@ -102,9 +109,9 @@
       <sensor type="gpu_lidar" name="gpu_lidar">
         <pose relative_to='laser_scan_frame'>0 0 0 0 0 0</pose>
-        <gz_frame_id>laser_scan_frame</gz_frame_id>
+        <gz_frame_id>${robot_name}/laser_scan_frame</gz_frame_id>
         <always_on>1</always_on>
         <visualize>true</visualize>
         <update_rate>100</update_rate>
-        <topic>scan</topic>
+        <topic>/${robot_name}/scan</topic>
         <ray>
           <scan>

Commit message: checkpoint 4

File: barista_robot_description/urdf/barista_robot_model.urdf.xacro (robot description, xacro)
@@ -4,4 +4,5 @@
 <xacro:arg name="robot_name" default="barista" />
 <xacro:arg name="use_controllers" default="false" />
+<xacro:property name="robot_name" value="$(arg robot_name)"/>
 <xacro:include filename="$(find barista_robot_description)/urdf/caster_wheel.xacro" />
 <xacro:include filename="$(find barista_robot_description)/urdf/cup_holder_tray.xacro" />
@@ -88,5 +89,5 @@
         <left_joint>joint_left_wheel</left_joint>
         <right_joint>joint_right_wheel</right_joint>
-        <wheel_separation>0.1</wheel_separation>
+        <wheel_separation>0.29</wheel_separation>
         <wheel_radius>0.035</wheel_radius>
         <topic>/$(arg robot_name)/cmd_vel</topic>
@@ -96,6 +97,6 @@
         <odom_topic>/$(arg robot_name)/odom</odom_topic>
         <tf_topic>/$(arg robot_name)/tf</tf_topic>
-        <frame_id>$(arg robot_name)/odom</frame_id>
-        <child_frame_id>$(arg robot_name)/base_link</child_frame_id>
+        <frame_id>/$(arg robot_name)/odom</frame_id>
+        <child_frame_id>/$(arg robot_name)/base_link</child_frame_id>
     </plugin>
 </gazebo>

File: barista_robot_description/urdf/drive_wheel.xacro (robot description, xacro)
@@ -16,5 +16,5 @@
         <origin rpy="0 1.5707 1.5707" xyz="0 0 0"/>
         <geometry>
-          <cylinder length="0.001" radius="0.035"/>
+          <cylinder length="0.03" radius="0.035"/>
         </geometry>
       </collision>
@@ -25,5 +25,4 @@
       </inertial>
     </link>
-    <!--
     <gazebo reference="${prefix}_wheel">
       <collision>
@@ -44,5 +43,4 @@
       </collision>
     </gazebo>
-    -->
     <joint name="joint_${prefix}_wheel" type="continuous">
       <origin rpy="0 0 0" xyz="0 ${y_offset} 0"/>

File: barista_robot_description/urdf/laser_scanner.xacro (robot description, xacro)
@@ -68,41 +68,4 @@
       <dynamics friction="0.01"/>
     </joint>
-    <!-- ros2_control hardware interface for the two actuated laser joints -->
-    <ros2_control name="GazeboSimSystem" type="system">
-      <hardware>
-        <plugin>gz_ros2_control/GazeboSimSystem</plugin>
-      </hardware>
-      <joint name="laser_scan_link_joint">
-        <command_interface name="position">
-          <param name="min">-0.05</param>
-          <param name="max">0.0</param>
-        </command_interface>
-        <state_interface name="position"/>
-        <state_interface name="velocity"/>
-        <state_interface name="effort"/>
-      </joint>
-      <joint name="laser_scan_model_link_joint">
-        <command_interface name="velocity">
-          <param name="min">0.0</param>
-          <param name="max">2.0</param>
-        </command_interface>
-        <state_interface name="position"/>
-        <state_interface name="velocity"/>
-        <state_interface name="effort"/>
-      </joint>
-    </ros2_control>
-    <gazebo>
-      <plugin filename="gz_ros2_control-system"
-              name="gz_ros2_control::GazeboSimROS2ControlPlugin">
-        <ros>
-          <namespace>/${robot_name}</namespace>
-          <!-- Some gz_ros2_control versions subscribe to the absolute
-               /robot_description topic even when namespaced; remap both
-               forms so each controller_manager gets its own robot. -->
-          <remapping>/robot_description:=/${robot_name}/robot_description</remapping>
-          <remapping>robot_description:=/${robot_name}/robot_description</remapping>
-        </ros>
-      </plugin>
-    </gazebo>
     <!-- GPU lidar sensor, publishing on /scan -->
     <gazebo reference="laser_scan_frame">

Commit message: Fix gazibo

File: barista_robot_description/urdf/barista_robot_model.urdf.xacro (robot description, xacro)
@@ -3,5 +3,5 @@
 <xacro:arg name="include_laser" default="true" />
 <xacro:arg name="robot_name" default="barista" />
-<xacro:arg name="use_controllers" default="false" />
+<xacro:arg name="robot_color" default="blue" />
 <xacro:property name="robot_name" value="$(arg robot_name)"/>
 <xacro:include filename="$(find barista_robot_description)/urdf/caster_wheel.xacro" />
@@ -35,12 +35,13 @@
     </visual>
     <collision>
+        <origin xyz="0 0 0.0775" rpy="0 0 0"/>
         <geometry>
-            <box size="0.1 0.1 0.1"/>
+            <cylinder length="0.155" radius="0.178"/>
         </geometry>
     </collision>
     <inertial>
         <mass value="0.5"/>
-        <origin rpy="0 0 0" xyz="0 0 0"/>
-        <inertia ixx="0.0008333333333333335" ixy="0" ixz="0" iyy="0.0008333333333333335" iyz="0" izz="0.0008333333333333335"/>
+        <origin rpy="0 0 0" xyz="0 0 0.0775"/>
+        <inertia ixx="0.00496" ixy="0" ixz="0" iyy="0.00496" iyz="0" izz="0.00792"/>
     </inertial>
 </link>
@@ -58,5 +59,5 @@
 <xacro:cup_holder_tray parent="base_link"/>
 <xacro:if value="$(arg include_laser)">
-    <xacro:laser_scanner parent="chassis" robot_name="$(arg robot_name)"/>
+    <xacro:laser_scanner parent="chassis" robot_name="${robot_name}"/>
 </xacro:if>
 <!-- ============================================================ -->
@@ -67,5 +68,5 @@
     <plugin filename="gz-sim-joint-state-publisher-system"
             name="gz::sim::systems::JointStatePublisher">
-        <topic>/$(arg robot_name)/joint_states</topic>
+        <topic>/${robot_name}/joint_states</topic>
         <update_rate>30</update_rate>
         <joint_name>joint_left_wheel</joint_name>
@@ -91,12 +92,12 @@
         <wheel_separation>0.29</wheel_separation>
         <wheel_radius>0.035</wheel_radius>
-        <topic>/$(arg robot_name)/cmd_vel</topic>
+        <topic>/${robot_name}/cmd_vel</topic>
         <publish_odom>true</publish_odom>
         <publish_odom_tf>true</publish_odom_tf>
         <publish_wheel_tf>true</publish_wheel_tf>
-        <odom_topic>/$(arg robot_name)/odom</odom_topic>
-        <tf_topic>/$(arg robot_name)/tf</tf_topic>
-        <frame_id>/$(arg robot_name)/odom</frame_id>
-        <child_frame_id>/$(arg robot_name)/base_link</child_frame_id>
+        <odom_topic>/${robot_name}/odom</odom_topic>
+        <tf_topic>/${robot_name}/tf</tf_topic>
+        <frame_id>${robot_name}/odom</frame_id>
+        <child_frame_id>${robot_name}/base_link</child_frame_id>
     </plugin>
 </gazebo>

Commit message: part1 cleanup

File: barista_robot_description/urdf/barista_robot_model.urdf.xacro (robot description, xacro)
@@ -54,5 +54,7 @@
 <!-- COMPONENT INSTANTIATION                                       -->
 <!-- ============================================================ -->
-<xacro:drive_wheels parent="chassis"/>
+<!-- <xacro:drive_wheels parent="chassis"/> -->
+<xacro:drive_wheel prefix="left" parent="chassis" y_offset="0.145" color="white"/>
+<xacro:drive_wheel prefix="right" parent="chassis" y_offset="-0.145" color="white"/>
 <xacro:caster_wheel prefix="front" parent="chassis" x_offset="0.178"/>
 <xacro:caster_wheel prefix="back"  parent="chassis" x_offset="-0.178"/>

File: barista_robot_description/urdf/drive_wheel.xacro (robot description, xacro)
@@ -4,5 +4,5 @@
        `parent` at y = y_offset (e.g. left: 0.145, right: -0.145).
        Material "red" must already be defined in the including file. -->
-  <xacro:macro name="drive_wheel" params="prefix parent y_offset">
+  <xacro:macro name="drive_wheel" params="prefix parent y_offset color">
     <link name="${prefix}_wheel">
       <visual>
@@ -11,5 +11,5 @@
           <cylinder length="0.0206" radius="0.0352"/>
         </geometry>
-        <material name="red"/>
+        <material name="${color}"/>
       </visual>
       <collision>

Commit message: Fix Robot Chase

File: barista_robot_description/urdf/barista_robot_model.urdf.xacro (robot description, xacro)
@@ -57,6 +57,6 @@
 <xacro:drive_wheel prefix="left" parent="chassis" y_offset="0.145" color="white"/>
 <xacro:drive_wheel prefix="right" parent="chassis" y_offset="-0.145" color="white"/>
-<xacro:caster_wheel prefix="front" parent="chassis" x_offset="0.178"/>
-<xacro:caster_wheel prefix="back"  parent="chassis" x_offset="-0.178"/>
+<xacro:caster_wheel prefix="front" parent="chassis" x_offset="0.143"/>
+<xacro:caster_wheel prefix="back"  parent="chassis" x_offset="-0.143"/>
 <xacro:cup_holder_tray parent="base_link"/>
 <xacro:if value="$(arg include_laser)">

File: barista_robot_description/urdf/caster_wheel.xacro (robot description, xacro)
@@ -33,5 +33,5 @@
       <child link="${prefix}_yaw"/>
       <limit effort="1000.0" velocity="100.0"/>
-      <dynamics damping="0.0" friction="0.1"/>
+      <dynamics damping="0.0" friction="0.0"/>
     </joint>
     <link name="${prefix}_roll">
@@ -61,5 +61,5 @@
       <parent link="${prefix}_yaw"/>
       <limit effort="1000.0" velocity="100.0"/>
-      <dynamics damping="0.0" friction="0.1"/>
+      <dynamics damping="0.0" friction="0.0"/>
     </joint>
     <link name="${prefix}_pitch">
@@ -74,12 +74,12 @@
         <origin rpy="0 1.5707 1.5707" xyz="0 0 0"/>
         <geometry>
-          <sphere radius="0.010"/>
+          <sphere radius="0.035"/>
         </geometry>
       </collision>
-      <inertial>
-        <origin rpy="0 1.5707 1.5707" xyz="0 0 0"/>
-        <mass value="0.001"/>
-        <inertia ixx="4e-08" ixy="0" ixz="0" iyy="4e-08" iyz="0" izz="4e-08"/>
-      </inertial>
+        <inertial>
+            <origin rpy="0 1.5707 1.5707" xyz="0 0 0"/>
+            <mass value="0.05"/>
+            <inertia ixx="2.5e-05" ixy="0" ixz="0" iyy="2.5e-05" iyz="0" izz="2.5e-05"/>
+        </inertial>
     </link>
     <joint name="${prefix}_pitch_joint" type="continuous">
@@ -89,6 +89,18 @@
       <parent link="${prefix}_roll"/>
       <limit effort="1000.0" velocity="100.0"/>
-      <dynamics damping="0.0" friction="0.1"/>
+      <dynamics damping="0.0" friction="0.0"/>
     </joint>
+    <gazebo reference="${prefix}_pitch">
+      <collision>
+        <surface>
+          <friction>
+            <ode>
+              <mu>0.05</mu>
+              <mu2>0.05</mu2>
+            </ode>
+          </friction>
+        </surface>
+      </collision>
+    </gazebo>
   </xacro:macro>
 </robot>

File: barista_robot_description/urdf/laser_scanner.xacro (robot description, xacro)
@@ -26,5 +26,5 @@
     </link>
     <joint name="laser_scan_link_joint" type="prismatic">
-      <origin rpy="0 0 0" xyz="0.160 0 0.155"/>
+      <origin rpy="0 0 0" xyz="0.140 0 0.155"/>
       <parent link="${parent}"/>
       <child link="laser_scan_link"/>
